File: Tarea 4 - Diseño PCB (2023-1283)/DRIVER-RS485.kicad_sch (KiCad schematic)
At the start: 1 part

Commit message: Actualizacion
Parts:
- added C15: C_0603, PCM_Capacitor_SMD_AKL:C_0603_1608Metric, symbol PCM_Capacitor_AKL:C_0603
- added D10: SM712, PCM_Package_TO_SOT_SMD_AKL:SOT-23, symbol PCM_Diode_TVS_AKL:SM712
Connections:
- net RS_485_A: now also C8.9 (A)
- net RS_485_B: now also C8.8 (B)
- net UART_IN: now also C8.3 (TXD)
- net UART_OUT: now also C8.4 (RXD)
- net +3.3V: now reaches C8.1 (VCC)
- net +3.3V: now also C15.1, D10.2 (A2)
- net GND: now reaches C8.2 (GND)
- net GND: now also C15.2, D10.1 (A1), D10.3 (Com)
- net GPIO_C: now reaches C8.5 (CON)
