File: Tarea 4 - Diseño PCB (2023-1283)/INPUT_NPN.kicad_sch (KiCad schematic)
At the start: 0 parts

Commit message: Actualizacion
Parts:
- added D1, D8: DL4007, PCM_Diode_SMD_AKL:D_MELF, symbol PCM_Diode_AKL:DL4007
- added OC1, OC5: LTV-357T-B, PCM_Package_SO_AKL:SO-4_4.4x3.9mm_P2.54mm, symbol PCM_Optocoupler_AKL:LTV-357T-B
- added R18, R19, R4, R5: R_0603, PCM_Resistor_SMD_AKL:R_0603_1608Metric, symbol PCM_Resistor_US_AKL:R_0603
Connections:
- new net: D8.1 (K), OC5.1, R18.1
- new net: D1.1 (K), OC1.1, R4.1
- new net +3.3V: R19.2, R5.2
- new net GND: D1.2 (A), D8.2 (A), OC1.2, OC1.3, OC5.2, OC5.3
- new net NPN_D_IMPUT_1: OC1.4, R5.1
- new net NPN_D_IMPUT_2: OC5.4, R19.1
- new net NPN_IN_1_: R4.2
- new net NPN_IN_2_: R18.2
