File: Tarea 4 - Diseño PCB (2023-1283)/INPUT_PNP.kicad_sch (KiCad schematic)
At the start: 0 parts

Commit message: Actualizacion
Parts:
- added D2, D9: DL4007, PCM_Diode_SMD_AKL:D_MELF, symbol PCM_Diode_AKL:DL4007
- added OC2, OC6: LTV-357T-B, PCM_Package_SO_AKL:SO-4_4.4x3.9mm_P2.54mm, symbol PCM_Optocoupler_AKL:LTV-357T-B
- added R25, R26, R6, R7: R_0603, PCM_Resistor_SMD_AKL:R_0603_1608Metric, symbol PCM_Resistor_US_AKL:R_0603
Connections:
- new net: OC6.3, R26.2
- new net: D2.1 (K), OC2.1, R6.1
- new net: OC2.3, R7.2
- new net: D9.1 (K), OC6.1, R25.1
- new net +3.3V: OC2.4, OC6.4
- new net GND: D2.2 (A), D9.2 (A), OC2.2, OC6.2, R26.1, R7.1
- new net PNP_IN_1_: R6.2
- new net PNP_IN_2_: R25.2
