File: Tarea 4 - Diseño PCB (2023-1283)/RLY_1.kicad_sch (KiCad schematic)
At the start: 0 parts

Commit message: Actualizacion
Parts:
- added K1, K2: SRA-24VDC-CL, Battery:RELAY-TH_SRA-X-CX, symbol RLY:SRA-24VDC-CL
- added U5: LK1802, Battery:LK1802, symbol RLY:LK1802
Connections:
- new net: K2.4, U5.6 (2C)
- new net: K1.4, U5.1 (1C)
- new net GND: U5.2 (E)
- new net ON_RLY_1: U5.3 (1B)
- new net ON_RLY_2: U5.4 (2B)
- new net RLY_COM_1: K1.5
- new net RLY_COM_2: K2.5
- new net RLY_NC_1: K1.2
- new net RLY_NC_2: K2.2
- new net RLY_NO_1: K1.1
- new net RLY_NO_2: K2.1
- new net VCC: K1.3, K2.3, U5.5 (COM)
