File: Tarea 4 - Diseño PCB (2023-1283)/Board_nivara_control.kicad_sch (KiCad schematic)
At the start: 3 parts, among them U1 ESP32-S3-WROOM-1

Commit message: Actualizacion
Parts:
- added R27: R_0603, PCM_Resistor_SMD_AKL:R_0603_1608Metric, symbol PCM_Resistor_US_AKL:R_0603
Connections:
- net +3.3V: now also R27.1
- net RUN/STOP: now also U1.30 (SPIDQS/GPIO37/FSPIQ/SUBSPIQ), R27.2
- net OUTPUT_NPN/NPN_IN_1_: now reaches U1.10 (GPIO17/U1TXD/ADC2_CH6)
- net OUTPUT_NPN/NPN_IN_2: now reaches U1.11 (GPIO18/U1RXD/ADC2_CH7/CLK_OUT3)
- net INPUT_PNP/PNP_D_IMPUT_2: now reaches U1.12 (GPIO8/TOUCH8/ADC1_CH7/SUBSPICS1)
- net Modulo RLY/ON_RLY_2: now reaches U1.15 (GPIO3/TOUCH3/ADC1_CH2)
- net MODULO_D_IN/D_INPUT_1: now reaches U1.17 (GPIO9/TOUCH9/ADC1_CH8/FSPIHD/SUBSPIHD)
- net MODULO_D_IN/D_INPUT_2: now reaches U1.18 (GPIO10/TOUCH10/ADC1_CH9/FSPICS0/FSPIIO4/SUBSPICS0)
- net INPUT_NPN/NPN_D_IMPUT_1: now reaches U1.19 (GPIO11/TOUCH11/ADC2_CH0/FSPID/FSPIIO5/SUBSPID)
- net INPUT_NPN/NPN_D_IMPUT_2: now reaches U1.20 (GPIO12/TOUCH12/ADC2_CH1/FSPICLK/FSPIIO6/SUBSPICLK)
- net MODULO_AOUT_0-10/SDA: now reaches U1.21 (GPIO13/TOUCH13/ADC2_CH2/FSPIQ/FSPIIO7/SUBSPIQ)
- net MODULO_AOUT_0-10/SCLK: now reaches U1.22 (GPIO14/TOUCH14/ADC2_CH3/FSPIWP/FSPIDQS/SUBSPIWP)
- net DRIVER-RS485/GPIO_C: now reaches U1.26 (GPIO45)
- net Modulo RLY/ON_RLY_1: now reaches U1.38 (GPIO2/TOUCH2/ADC1_CH1)
- net MODULO_ 0-32V_IN/D_0-32V: now reaches U1.39 (GPIO1/TOUCH1/ADC1_CH0)
- net Modulo A_420_IN/A_420_OUT: now reaches U1.4 (GPIO4/TOUCH4/ADC1_CH3)
- net MODULO_0-10V_IN/D_0-10V: now reaches U1.6 (GPIO6/TOUCH6/ADC1_CH5)
- net INPUT_PNP/PNP_D_IMPUT_1: now reaches U1.7 (GPIO7/TOUCH7/ADC1_CH6)
Other:
- sheet RLY_1 renamed Modulo RLY
- removed sheet RLY_2
- added sheet MODULO_ 0-32V_IN (MODULO_ 0-32V_IN.kicad_sch)
- added sheet MODULO_0-10V_IN (untitled.kicad_sch)
- added sheet MODULO_AOUT_0-10 (MODULO_AOUT_0-10.kicad_sch)
- added sheet MODULO_AOUT_420 (MODULO_AOUT_420.kicad_sch)
- added sheet MODULO_D_IN (MODULO_D_IN.kicad_sch)
- added sheet Modulo A_420_IN (Modulo A_420_IN.kicad_sch)
- sheet DRIVER-RS485 ports: added GPIO_C; removed none
- sheet INPUT_NPN ports: added NPN_D_IMPUT_1, NPN_D_IMPUT_2, NPN_IN_1_, NPN_IN_2_; removed none
- sheet INPUT_PNP ports: added PNP_D_IMPUT_1, PNP_D_IMPUT_2, PNP_IN_1_, PNP_IN_2_; removed none
- sheet Modulo RLY ports: added ON_RLY_1, ON_RLY_2, RLY_COM_1, RLY_COM_2, RLY_NC_1, RLY_NC_2, RLY_NO_1, RLY_NO_2; removed none
- sheet OUTPUT_NPN ports: added DOUT_NPN_1, DOUT_NPN_2, NPN_IN_1_, NPN_IN_2; removed none

Commit message: New Actualizacion
Parts:
- added R32, R33: R_0603, PCM_Resistor_SMD_AKL:R_0603_1608Metric, symbol PCM_Resistor_US_AKL:R_0603
Connections:
- net +3.3V: now also R32.2, R33.2
- net MODULO_AOUT_0-10/SDA: now also R32.1, R33.1

Commit message: Complete
Connections:
- net OUTPUT_PNP/PNP_1: now reaches U1.23 (GPIO21)
- net OUTPUT_PNP/PNP_2: now reaches U1.31 (GPIO38/FSPIWP/SUBSPIWP)
- net OUTPUT_NPN/NPN_IN_1_ renamed OUTPUT_NPN/NPN_1
- net OUTPUT_NPN/NPN_IN_2 renamed OUTPUT_NPN/NPN_2
Other:
- sheet OUTPUT_NPN ports: added NPN_1, NPN_2, NPN_OUT_1, NPN_OUT_2; removed DOUT_NPN_1, DOUT_NPN_2, NPN_IN_1_, NPN_IN_2
- sheet OUTPUT_PNP ports: added PNP_1, PNP_2, PNP_OUT_1, PNP_OUT_2; removed none
Changed lines of the file:
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@@
+	(wire
+		(pts
+			(xy 308.61 184.15) (xy 311.15 184.15)
+		)
+		(stroke
+			(width 0)
+			(type default)
+		)
+	)
 	(wire
 		(pts
@@
 	(wire
 		(pts
+			(xy 262.89 181.61) (xy 285.75 181.61)
+		)
+		(stroke
+			(width 0)
+			(type default)
+		)
+	)
+	(wire
+		(pts
 			(xy 270.51 166.37) (xy 270.51 91.44)
 		)
@@
 	(wire
 		(pts
+			(xy 261.62 99.06) (xy 256.54 99.06)
+		)
+		(stroke
+			(width 0)
+			(type default)
+		)
+	)
+	(wire
+		(pts
 			(xy 259.08 44.45) (xy 259.08 55.88)
 		)
@@
 	(wire
 		(pts
+			(xy 308.61 181.61) (xy 311.15 181.61)
+		)
+		(stroke
+			(width 0)
+			(type default)
+		)
+	)
+	(wire
+		(pts
 			(xy 295.91 29.21) (xy 297.18 29.21)
 		)
@@
 	(wire
 		(pts
+			(xy 256.54 96.52) (xy 262.89 96.52)
+		)
+		(stroke
+			(width 0)
+			(type default)
+		)
+	)
+	(wire
+		(pts
 			(xy 259.08 55.88) (xy 256.54 55.88)
 		)
@@
 	(wire
 		(pts
+			(xy 262.89 96.52) (xy 262.89 181.61)
+		)
+		(stroke
+			(width 0)
+			(type default)
+		)
+	)
+	(wire
+		(pts
 			(xy 306.07 68.58) (xy 311.15 68.58)
 		)
@@
 		(pts
 			(xy 285.75 101.6) (xy 279.4 101.6)
+		)
+		(stroke
+			(width 0)
+			(type default)
+		)
+	)
+	(wire
+		(pts
+			(xy 285.75 184.15) (xy 261.62 184.15)
+		)
+		(stroke
+			(width 0)
+			(type default)
+		)
+	)
+	(wire
+		(pts
+			(xy 261.62 184.15) (xy 261.62 99.06)
 		)
 		(stroke
@@
 	(hierarchical_label "DOUT_PNP_2"
 		(shape output)
-		(at 311.15 185.42 0)
+		(at 311.15 184.15 0)
 		(effects
 			(font
@@
 	)
 	(sheet
-		(at 285.75 177.8)
-		(size 22.86 12.7)
+		(at 285.75 180.34)
+		(size 22.86 6.35)
 		(exclude_from_sim no)
 		(in_bom yes)
@@
 		)
 		(property "Sheetname" "OUTPUT_PNP"
-			(at 285.75 177.0884 0)
+			(at 285.75 179.6284 0)
 			(effects
 				(font
@@
 		)
 		(property "Sheetfile" "OUTPUT_PNP.kicad_sch"
-			(at 285.75 191.0846 0)
+			(at 285.75 187.2746 0)
 			(effects
 				(font
@@
 				(justify left top)
 				(hide yes)
+			)
+		)
+		(pin "PNP_1" output
+			(at 285.75 181.61 180)
+			(effects
+				(font
+					(size 1.27 1.27)
+				)
+				(justify left)
+			)
+		)
+		(pin "PNP_2" output
+			(at 285.75 184.15 180)
+			(effects
+				(font
+					(size 1.27 1.27)
+				)
+				(justify left)
+			)
+		)
+		(pin "PNP_OUT_1" output
+			(at 308.61 181.61 0)
+			(effects
+				(font
+					(size 1.27 1.27)
+				)
+				(justify right)
+			)
+		)
+		(pin "PNP_OUT_2" output
+			(at 308.61 184.15 0)
+			(effects
+				(font
+					(size 1.27 1.27)
+				)
+				(justify right)
 			)
 		)
@@
 	(sheet
 		(at 281.94 163.83)
-		(size 29.21 11.43)
+		(size 29.21 8.89)
 		(exclude_from_sim no)
 		(in_bom yes)
@@
 		)
 		(property "Sheetfile" "OUTPUT_NPN.kicad_sch"
-			(at 281.94 175.8446 0)
+			(at 281.94 173.3046 0)
 			(effects
 				(font
@@
 			)
 		)
-		(pin "DOUT_NPN_1" output
+		(pin "NPN_1" output
+			(at 281.94 166.37 180)
+			(effects
+				(font
+					(size 1.27 1.27)
+				)
+				(justify left)
+			)
+		)
+		(pin "NPN_2" output
+			(at 281.94 170.18 180)
+			(effects
+				(font
+					(size 1.27 1.27)
+				)
+				(justify left)
+			)
+		)
+		(pin "NPN_OUT_1" output
 			(at 311.15 166.37 0)
 			(effects
@@
 			)
 		)
-		(pin "NPN_IN_1_" input
-			(at 281.94 166.37 180)
-			(effects
-				(font
-					(size 1.27 1.27)
-				)
-				(justify left)
-			)
-		)
-		(pin "NPN_IN_2" input
-			(at 281.94 170.18 180)
-			(effects
-				(font
-					(size 1.27 1.27)
-				)
-				(justify left)
-			)
-		)
-		(pin "DOUT_NPN_2" output
+		(pin "NPN_OUT_2" output
 			(at 311.15 170.18 0)
 			(effects
