File: Tarea 4 - Diseño PCB (2023-1283)/OUTPUT_PNP.kicad_sch (KiCad schematic)
At the start: 0 parts

Commit message: Complete
Parts:
- added R34, R35: R_0603, PCM_Resistor_SMD_AKL:R_0603_1608Metric, symbol PCM_Resistor_US_AKL:R_0603
- added U6, U7: GAQY211G2S, Battery:GQRLY, symbol RLY:GAQY211G2S
Connections:
- new net: R34.1, U6.1
- new net: R35.1, U7.1
- new net GND: U6.2, U7.2
- new net PNP_1: R34.2
- new net PNP_2: R35.2
- new net PNP_OUT_1: U6.3
- new net PNP_OUT_2: U7.3
- new net VCC: U6.4, U7.4
