File: Tarea 4 - Diseño PCB (2023-1283)/Tarea 4 - Diseño PCB (2023-1283).kicad_pcb (KiCad board)
At the start: 2 copper layers, 28 parts, among them J1 Screw_Terminal_2_P5.00mm, J10 Screw_Terminal_4_P5.00mm, J12 Screw_Terminal_2_P5.00mm, J2 Screw_Terminal_4_P5.00mm, J3 Screw_Terminal_2_P5.00mm, J4 Screw_Terminal_2_P5.00mm, J6 Screw_Terminal_3_P5.00mm, J7 Screw_Terminal_3_P5.00mm, J8 Screw_Terminal_2_P5.00mm, J9 Screw_Terminal_6_P5.00mm, U1 ESP32-S3-WROOM-1, U2 AP63203WU

Commit message: Actualizacion
Parts:
- removed J4: Screw_Terminal_2_P5.00mm, TerminalBlock_Phoenix:TerminalBlock_Phoenix_PT-1,5-2-5.0-H_1x02_P5.00mm_Horizontal
- added C10: C_0805, PCM_Capacitor_SMD_AKL:C_0805_2012Metric, F.Cu at (41.0, 154.7)
- added C11: C_0805, PCM_Capacitor_SMD_AKL:C_0805_2012Metric, F.Cu at (72.4, 133.5)
- added C12: C_0805, PCM_Capacitor_SMD_AKL:C_0805_2012Metric, F.Cu at (72.4, 136.6)
- added C13: C_0805, PCM_Capacitor_SMD_AKL:C_0805_2012Metric, F.Cu at (83.4, 133.4)
- added C14: C_0805, PCM_Capacitor_SMD_AKL:C_0805_2012Metric, F.Cu at (83.4, 136.6)
- added C15: C_0603, PCM_Capacitor_SMD_AKL:C_0603_1608Metric, F.Cu at (34.0, 159.2)
- added C7: C_0805, PCM_Capacitor_SMD_AKL:C_0805_2012Metric, F.Cu at (85.0, 160.5)
- added C9: C_0805, PCM_Capacitor_SMD_AKL:C_0805_2012Metric, F.Cu at (72.2, 160.5)
- added D1: DL4007, PCM_Diode_SMD_AKL:D_MELF, F.Cu at (39.7, 143.1)
- added D10: SM712, PCM_Package_TO_SOT_SMD_AKL:SOT-23, F.Cu at (34.2, 155.4)
- added D2: DL4007, PCM_Diode_SMD_AKL:D_MELF, F.Cu at (63.8, 113.8)
- added D3: MB24F_C7427849, Battery:MB24F, F.Cu at (79.6, 158.0)
- added D4: MB24F_C7427849, Battery:MB24F, F.Cu at (66.7, 158.0)
- added D5: DL4007, PCM_Diode_SMD_AKL:D_MELF, F.Cu at (83.8, 113.8)
- added D6: DL4007, PCM_Diode_SMD_AKL:D_MELF, F.Cu at (83.8, 119.1)
- added D7: SMF24A, PCM_Diode_SMD_AKL:D_SOD-123F, F.Cu at (66.6, 134.1)
- added D8: DL4007, PCM_Diode_SMD_AKL:D_MELF, F.Cu at (39.7, 148.4)
- added D9: DL4007, PCM_Diode_SMD_AKL:D_MELF, F.Cu at (63.8, 119.1)
- added J5: Screw_Terminal_4_P5.00mm, TerminalBlock_Phoenix:TerminalBlock_Phoenix_PT-1,5-4-5.0-H_1x04_P5.00mm_Horizontal, F.Cu at (189.5, 43.5)
- added K1: SRA-24VDC-CL, Battery:RELAY-TH_SRA-X-CX, F.Cu at (144.0, 157.3)
- added K2: SRA-24VDC-CL, Battery:RELAY-TH_SRA-X-CX, F.Cu at (129.0, 157.3)
- added OC1: LTV-357T-B, PCM_Package_SO_AKL:SO-4_4.4x3.9mm_P2.54mm, F.Cu at (30.7, 132.5)
- added OC2: LTV-357T-B, PCM_Package_SO_AKL:SO-4_4.4x3.9mm_P2.54mm, F.Cu at (54.7, 103.2)
- added OC3: LTV-357T-B, PCM_Package_SO_AKL:SO-4_4.4x3.9mm_P2.54mm, F.Cu at (74.8, 103.2)
- added OC4: LTV-357T-B, PCM_Package_SO_AKL:SO-4_4.4x3.9mm_P2.54mm, F.Cu at (74.8, 108.9)
- added OC5: LTV-357T-B, PCM_Package_SO_AKL:SO-4_4.4x3.9mm_P2.54mm, F.Cu at (30.7, 138.2)
- added OC6: LTV-357T-B, PCM_Package_SO_AKL:SO-4_4.4x3.9mm_P2.54mm, F.Cu at (54.7, 108.9)
- added R10: R_0603, PCM_Resistor_SMD_AKL:R_0603_1608Metric, F.Cu at (71.8, 154.9)
- added R11: R_0603, PCM_Resistor_SMD_AKL:R_0603_1608Metric, F.Cu at (71.8, 157.6)
- added R12: R_0603, PCM_Resistor_SMD_AKL:R_0603_1608Metric, F.Cu at (40.6, 157.6)
- added R13: R_0603, PCM_Resistor_SMD_AKL:R_0603_1608Metric, F.Cu at (81.8, 101.7)
- added R14: R_0603, PCM_Resistor_SMD_AKL:R_0603_1608Metric, F.Cu at (81.8, 104.4)
- added R15: R_0603, PCM_Resistor_SMD_AKL:R_0603_1608Metric, F.Cu at (81.8, 107.1)
- added R16: R_0603, PCM_Resistor_SMD_AKL:R_0603_1608Metric, F.Cu at (81.8, 109.8)
- added R17: R_0603, PCM_Resistor_SMD_AKL:R_0603_1608Metric, F.Cu at (72.0, 125.2)
- added R18: R_0603, PCM_Resistor_SMD_AKL:R_0603_1608Metric, F.Cu at (37.7, 136.4)
- added R19: R_0603, PCM_Resistor_SMD_AKL:R_0603_1608Metric, F.Cu at (37.7, 139.1)
- added R20: R_0603, PCM_Resistor_SMD_AKL:R_0603_1608Metric, F.Cu at (78.9, 125.2)
- added R21: R_0603, PCM_Resistor_SMD_AKL:R_0603_1608Metric, F.Cu at (78.9, 127.9)
- added R22: R_0603, PCM_Resistor_SMD_AKL:R_0603_1608Metric, F.Cu at (78.9, 130.6)
- added R23: R_0603, PCM_Resistor_SMD_AKL:R_0603_1608Metric, F.Cu at (72.0, 127.9)
- added R24: R_0603, PCM_Resistor_SMD_AKL:R_0603_1608Metric, F.Cu at (72.0, 130.6)
- added R25: R_0603, PCM_Resistor_SMD_AKL:R_0603_1608Metric, F.Cu at (61.8, 107.1)
- added R26: R_0603, PCM_Resistor_SMD_AKL:R_0603_1608Metric, F.Cu at (61.8, 109.8)
- added R27: R_0603, PCM_Resistor_SMD_AKL:R_0603_1608Metric, F.Cu at (27.8, 154.4)
- added R28: R_0603, PCM_Resistor_SMD_AKL:R_0603_1608Metric, F.Cu at (51.8, 152.6)
- added R32: R_0603, PCM_Resistor_SMD_AKL:R_0603_1608Metric, F.Cu at (27.8, 157.2)
- added R33: R_0603, PCM_Resistor_SMD_AKL:R_0603_1608Metric, F.Cu at (27.8, 159.9)
- added R34: R_0603, PCM_Resistor_SMD_AKL:R_0603_1608Metric, F.Cu at (51.8, 135.2)
- added R35: R_0603, PCM_Resistor_SMD_AKL:R_0603_1608Metric, F.Cu at (51.8, 137.9)
- added R36: R_0603, PCM_Resistor_SMD_AKL:R_0603_1608Metric, F.Cu at (51.8, 155.3)
- added R4: R_0603, PCM_Resistor_SMD_AKL:R_0603_1608Metric, F.Cu at (37.7, 131.0)
- added R5: R_0603, PCM_Resistor_SMD_AKL:R_0603_1608Metric, F.Cu at (37.7, 133.7)
- added R6: R_0603, PCM_Resistor_SMD_AKL:R_0603_1608Metric, F.Cu at (61.8, 101.7)
- added R7: R_0603, PCM_Resistor_SMD_AKL:R_0603_1608Metric, F.Cu at (61.8, 104.4)
- added R8: R_0603, PCM_Resistor_SMD_AKL:R_0603_1608Metric, F.Cu at (84.7, 154.9)
- added R9: R_0603, PCM_Resistor_SMD_AKL:R_0603_1608Metric, F.Cu at (84.7, 157.6)
- added U3: GP8201-SOP8, Battery:GP8201, F.Cu at (66.9, 127.9)
- added U4: GP8303-TC50-EW, Battery:GP8303, F.Cu at (84.1, 127.8)
- added U5: LK1802, Battery:LK1802, F.Cu at (45.4, 102.5)
- added U6: GAQY211G2S, Battery:GQRLY, F.Cu at (53.0, 128.8)
- added U7: GAQY211G2S, Battery:GQRLY, F.Cu at (58.9, 128.8)
- added U8: GAQY211G2S, Battery:GQRLY, F.Cu at (53.0, 146.2)
- added U9: GAQY211G2S, Battery:GQRLY, F.Cu at (58.9, 146.2)
- moved TP1 131.6 mm to (177.0, 158.1)
- moved TP2 131.6 mm to (177.0, 161.5)
- moved TP4 130.5 mm to (183.0, 160.0)
- moved TP3 129.0 mm to (182.0, 155.5)
- moved JP1 120.0 mm to (177.7, 154.0)
- moved C3 116.1 mm to (182.0, 145.0)
- moved C4 116.1 mm to (182.1, 148.0)
- moved R2 114.4 mm to (177.7, 151.0)
- moved C6 111.8 mm to (177.8, 148.0)
- moved C1 110.7 mm to (185.5, 131.0)
- moved R3 108.8 mm to (177.8, 145.0)
- moved J8 90.2 mm to (201.5, 43.5), turned to 180 degrees
- moved J1 85.7 mm to (133.5, 43.5), turned to 180 degrees
- moved J7 82.5 mm to (144.5, 115.5)
- moved C2 81.9 mm to (182.5, 151.5)
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Connections:
- net /Board_nivara_control/RLY1_C renamed /RLY1_C
- net /Board_nivara_control/RLY2_C renamed /RLY2_C
- C8 pad 1: unconnected-(C8-VCC-Pad1) -> +3.3V
- C8 pad 2: unconnected-(C8-GND-Pad2) -> GND
- C8 pad 3: unconnected-(C8-TXD-Pad3) -> /Board_nivara_control/DRIVER-RS485/UART_IN
- C8 pad 4: unconnected-(C8-RXD-Pad4) -> /Board_nivara_control/DRIVER-RS485/UART_OUT
- C8 pad 5: unconnected-(C8-CON-Pad5) -> /Board_nivara_control/DRIVER-RS485/GPIO_C
- C8 pad 8: unconnected-(C8-B-Pad8) -> /Board_nivara_control/RS485-B
- C8 pad 9: unconnected-(C8-A-Pad9) -> /Board_nivara_control/RS485-A
- U1 pad 10: unconnected-(U1-GPIO17/U1TXD/ADC2_CH6-Pad10) -> /Board_nivara_control/OUTPUT_NPN/NPN_1
- U1 pad 11: unconnected-(U1-GPIO18/U1RXD/ADC2_CH7/CLK_OUT3-Pad11) -> /Board_nivara_control/OUTPUT_NPN/NPN_2
- U1 pad 12: unconnected-(U1-GPIO8/TOUCH8/ADC1_CH7/SUBSPICS1-Pad12) -> +3.3V
- U1 pad 15: unconnected-(U1-GPIO3/TOUCH3/ADC1_CH2-Pad15) -> /Board_nivara_control/Modulo RLY/ON_RLY_2
- U1 pad 17: unconnected-(U1-GPIO9/TOUCH9/ADC1_CH8/FSPIHD/SUBSPIHD-Pad17) -> /Board_nivara_control/MODULO_D_IN/D_INPUT_1
- U1 pad 18: unconnected-(U1-GPIO10/TOUCH10/ADC1_CH9/FSPICS0/FSPIIO4/SUBSPICS0-Pad18) -> /Board_nivara_control/MODULO_D_IN/D_INPUT_2
- U1 pad 19: unconnected-(U1-GPIO11/TOUCH11/ADC2_CH0/FSPID/FSPIIO5/SUBSPID-Pad19) -> /Board_nivara_control/INPUT_NPN/NPN_D_IMPUT_1
- U1 pad 20: unconnected-(U1-GPIO12/TOUCH12/ADC2_CH1/FSPICLK/FSPIIO6/SUBSPICLK-Pad20) -> /Board_nivara_control/INPUT_NPN/NPN_D_IMPUT_2
- U1 pad 21: unconnected-(U1-GPIO13/TOUCH13/ADC2_CH2/FSPIQ/FSPIIO7/SUBSPIQ-Pad21) -> /Board_nivara_control/MODULO_AOUT_0-10/SDA
- U1 pad 22: unconnected-(U1-GPIO14/TOUCH14/ADC2_CH3/FSPIWP/FSPIDQS/SUBSPIWP-Pad22) -> /Board_nivara_control/MODULO_AOUT_0-10/SCLK
- U1 pad 23: unconnected-(U1-GPIO21-Pad23) -> /Board_nivara_control/OUTPUT_PNP/PNP_1
- U1 pad 26: unconnected-(U1-GPIO45-Pad26) -> /Board_nivara_control/DRIVER-RS485/GPIO_C
- U1 pad 30: unconnected-(U1-SPIDQS/GPIO37/FSPIQ/SUBSPIQ-Pad30) -> /Board_nivara_control/RUN/STOP
- U1 pad 31: unconnected-(U1-GPIO38/FSPIWP/SUBSPIWP-Pad31) -> /Board_nivara_control/OUTPUT_PNP/PNP_2
- U1 pad 38: unconnected-(U1-GPIO2/TOUCH2/ADC1_CH1-Pad38) -> /Board_nivara_control/Modulo RLY/ON_RLY_1
- U1 pad 39: unconnected-(U1-GPIO1/TOUCH1/ADC1_CH0-Pad39) -> /Board_nivara_control/MODULO_ 0-32V_IN/D_0-32V
- U1 pad 4: unconnected-(U1-GPIO4/TOUCH4/ADC1_CH3-Pad4) -> /Board_nivara_control/A420_IN_1
- U1 pad 6: unconnected-(U1-GPIO6/TOUCH6/ADC1_CH5-Pad6) -> /Board_nivara_control/MODULO_0-10V_IN/D_0-10V
- U1 pad 7: unconnected-(U1-GPIO7/TOUCH7/ADC1_CH6-Pad7) -> +3.3V

Commit message: Actualizacion
Parts:
- moved C10 161.9 mm to (167.3, 53.3)
- moved R12 161.9 mm to (166.9, 56.3)
- moved D1 141.4 mm to (150.5, 55.2), turned to 90 degrees
- moved C12 140.9 mm to (212.1, 117.8), turned to 90 degrees
- moved D8 140.9 mm to (151.1, 62.2)
- moved R17 140.7 mm to (211.6, 107.3)
- moved R23 140.6 mm to (211.6, 110.5)
- moved R24 140.5 mm to (211.6, 113.7)
- moved U3 140.0 mm to (205.7, 110.5)
- moved D7 139.4 mm to (205.0, 117.5), turned to -90 degrees
- moved R28 138.6 mm to (181.5, 103.5)
- moved R36 138.6 mm to (181.5, 106.2)
- moved U8 138.6 mm to (182.6, 97.2)
- moved U9 138.6 mm to (188.6, 97.2)
- moved C11 137.4 mm to (208.9, 117.8), turned to -90 degrees
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
Commit message: NEW UPDATE
Parts:
- moved D2 36.3 mm to (176.5, 59.1)
- moved C14 19.5 mm to (209.7, 66.7)
- moved C13 18.6 mm to (205.1, 62.2)
- moved R1 15.6 mm to (193.7, 73.0)
- moved D9 13.1 mm to (153.0, 73.7)
- moved R28 12.8 mm to (193.0, 98.0), turned to 90 degrees
- moved R36 11.6 mm to (192.4, 102.4), turned to -90 degrees
- moved R14 10.9 mm to (193.7, 57.1)
- moved R16 10.8 mm to (193.5, 60.3)
- moved C1 10.6 mm to (120.0, 107.3)
- moved D6 9.84 mm to (176.5, 64.8)
- moved OC3 9.53 mm to (186.7, 52.7)
- moved R20 7.86 mm to (193.7, 63.5)
- moved U4 7.64 mm to (201.7, 66.8), turned to -90 degrees
- moved R21 7.41 mm to (193.7, 66.7)
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